File: saikoutype_nkbm-st110r2/pcb/NKBM-ST110r2.kicad_pcb (KiCad board)
At the start: 2 copper layers, 426.8 x 121.9 mm, 266 parts, among them K001 CHRY_MX, K021 CHRY_MX, K031 CHRY_MX, K041 CHRY_MX, K051 CHRY_MX, K061 CHRY_MX, K071 CHRY_MX, K081 CHRY_MX, K091 CHRY_MX, K0B1 CHRY_MX, K0C1 CHRY_MX, K0D1 CHRY_MX, K0E1 CHRY_MX, K101 CHRY_MX, K111 CHRY_MX, K121 CHRY_MX, K131 CHRY_MX, K141 CHRY_MX, K151 CHRY_MX, K161 CHRY_MX, K171 CHRY_MX, K181 CHRY_MX, K191 CHRY_MX, K1A1 CHRY_MX, K1B1 CHRY_MX, K1C1 CHRY_MX, K1D1 CHRY_MX, K1E1 CHRY_MX, K1E2 CHRY_MX, K201 CHRY_MX, K211 CHRY_MX, K221 CHRY_MX, K231 CHRY_MX, K241 CHRY_MX, K251 CHRY_MX, K261 CHRY_MX, K271 CHRY_MX, K281 CHRY_MX, K291 CHRY_MX, K2A1 CHRY_MX, K2B1 CHRY_MX, K2C1 CHRY_MX, K301 CHRY_MX, K311 CHRY_MX, K321 CHRY_MX, K331 CHRY_MX, K341 CHRY_MX, K351 CHRY_MX, K361 CHRY_MX, K371 CHRY_MX, K381 CHRY_MX, K391 CHRY_MX, K3A1 CHRY_MX, K3B1 CHRY_MX, K3C1 CHRY_MX, K3C2 CHRY_MX, K3E1 CHRY_MX, K3E2 CHRY_MX, K401 CHRY_MX, K402 CHRY_MX, K411 CHRY_MX, K421 CHRY_MX, K431 CHRY_MX, K441 CHRY_MX, K451 CHRY_MX, K461 CHRY_MX, K471 CHRY_MX, K481 CHRY_MX, K491 CHRY_MX, K4A1 CHRY_MX, K4B1 CHRY_MX, K4C1 CHRY_MX, K4D1 CHRY_MX, K4D2 CHRY_MX, K501 CHRY_MX, K511 CHRY_MX, K512 CHRY_MX, K521 CHRY_MX, K522 CHRY_MX, K531 CHRY_MX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

Commit message: Complete reannotation of schematic and PCB.
Parts:
- removed LOGO COPPER: SAIKOUTYPE110, Desktop:saikotypeNKBM-ST110r2reverse1
- added MODEL: NKBM-ST110_r2.0_18.02.11, null_keyboard:nkbm-st110_18.02, F.Cu at (335.4, 86.3)
- EXPANSION: renamed from GND; value EXP -> HEADER
- RESET: renamed from GND; value 2 pin header -> HEADER
- SPI: renamed from MISO; value SPI -> HEADER
- VCCIN: renamed from GND; value 5v -> HEADER
- renumbered D001 to D00, D021 to D02, D031 to D03, D041 to D04, D051 to D05, D061 to D06, D071 to D07, D081 to D08, D091 to D09, D0B1 to D0B, D0C1 to D0C, D0D1 to D0D, D0E1 to D0E, D101 to D10, D111 to D11, D121 to D12, D131 to D13, D141 to D14, D151 to D15, D161 to D16, D171 to D17, D181 to D18, D191 to D19, D1A1 to D1A, D1B1 to D1B, D1C1 to D1C, D1D1 to D1D, D1E1 to D1E, D201 to D20, D211 to D21, D221 to D22, D231 to D23, D241 to D24, D251 to D25, D261 to D26, D271 to D27, D281 to D28, D291 to D29, D2A1 to D2A, D2B1 to D2B, D2C1 to D2C, D301 to D30, D311 to D31, D321 to D32, D331 to D33, D341 to D34, D351 to D35, D361 to D36, D371 to D37, D381 to D38, D391 to D39, D3A1 to D3A, D3B1 to D3B, D3C1 to D3C, D3E1 to D3E, D401 to D40, D411 to D41, D421 to D42, D431 to D43, D441 to D44, D451 to D45, D461 to D46, D471 to D47, D481 to D48, D491 to D49, D4A1 to D4A, D4B1 to D4B, D4C1 to D4C, D4D1 to D4D, D501 to D50, D511 to D51, D521 to D52, D531 to D53, D541 to D54, D551 to D55, D561 to D56, D581 to D58, D591 to D59, D5A1 to D5A, D5D1 to D5D, D5E1 to D5E, D601 to D60, D611 to D61, D621 to D62, D631 to D63, D641 to D64, D651 to D65, D661 to D66, D671 to D67, D681 to D68, D691 to D69, D6A1 to D6A, D6B1 to D6B, D6C1 to D6C, D6D1 to D6D, D6E1 to D6E, D701 to D70, D711 to D71, D721 to D72, D731 to D73, D741 to D74, D751 to D75, D761 to D76, D771 to D77, D781 to D78, D791 to D79, D7A1 to D7A, D7B1 to D7B, D7C1 to D7C, D7D1 to D7D, D7E1 to D7E, K001 to K00, K021 to K02, K031 to K03, K041 to K04, K051 to K05, K061 to K06, K071 to K07, K081 to K08, K091 to K09, K0B1 to K0B, K0C1 to K0C, K0D1 to K0D, K0E1 to K0E, K101 to K10, K111 to K11, K121 to K12, K131 to K13, K141 to K14, K151 to K15, K161 to K16, K171 to K17, K181 to K18, K191 to K19, K1A1 to K1A, K1B1 to K1B, K1C1 to K1C, K1D1 to K1D, K1E1 to K1E, K201 to K20, K211 to K21, K221 to K22, K231 to K23, K241 to K24, K251 to K25, K261 to K26, K271 to K27, K281 to K28, K291 to K29, K2A1 to K2A, K2B1 to K2B, K2C1 to K2C, K301 to K30, K311 to K31, K321 to K32, K331 to K33, K341 to K34, K351 to K35, K361 to K36, K371 to K37, K381 to K38, K391 to K39, K3A1 to K3A, K3B1 to K3B, K3C1 to K3C, K3C2 to K3C, K3E1 to K3E, K401 to K40, K411 to K41, K421 to K42, K431 to K43, K441 to K44, K451 to K45, K461 to K46, K471 to K47, K481 to K48, K491 to K49, K4A1 to K4A, K4B1 to K4B, K4C1 to K4C, K4D1 to K4D, K501 to K50, K511 to K51, K512 to K511, K521 to K52, K522 to K521, K531 to K53, K541 to K54, K543 to K541, K551 to K55, K554 to K551, K571 to K57, K581 to K58, K591 to K59, K592 to K591, K5A1 to K5A, K5A2 to K5A1, K5D1 to K5D, K5D2 to K5D1, K5E1 to K5E, K601 to K60, K611 to K61, K621 to K62, K631 to K63, K641 to K64, K651 to K65, K661 to K66, K671 to K67, K681 to K68, K691 to K69, K6A1 to K6A, K6B1 to K6B, K6C1 to K6C, K6D1 to K6D, K6E1 to K6E, K701 to K70, K711 to K71, K721 to K72, K731 to K73, K741 to K74, K751 to K75, K761 to K76, K771 to K77, K781 to K78, K791 to K79, K7A1 to K7A, K7B1 to K7B, K7C1 to K7C, K7D1 to K7D, K7E1 to K7E, L01 to L00, L11 to L01, L21 to L02, L31 to L03, L41 to L04, L51 to L05, L61 to L06, L71 to L07, L81 to L08, L91 to L09, R01 to R00, R11 to R01, R21 to R02, R31 to R03, R41 to R04, R51 to R05, R61 to R06, R71 to R07, R81 to R08, R91 to R09
Routing:
- net /GND: track 815.7 -> 831.9 mm
Other:
- net class /GND: trace_width 2 -> 1
- net class Default: trace_width 2 -> 1
