File: saikoutype_nkbm-st110r2/pcb/NKBM-ST110r2.kicad_pcb (KiCad board)
At the start: 2 copper layers, 426.8 x 121.9 mm, 266 parts, among them K00 CHRY_MX, K02 CHRY_MX, K03 CHRY_MX, K04 CHRY_MX, K05 CHRY_MX, K06 CHRY_MX, K07 CHRY_MX, K08 CHRY_MX, K09 CHRY_MX, K0B CHRY_MX, K0C CHRY_MX, K0D CHRY_MX, K0E CHRY_MX, K10 CHRY_MX, K11 CHRY_MX, K12 CHRY_MX, K13 CHRY_MX, K14 CHRY_MX, K15 CHRY_MX, K16 CHRY_MX, K17 CHRY_MX, K18 CHRY_MX, K19 CHRY_MX, K1A CHRY_MX, K1B CHRY_MX, K1C CHRY_MX, K1D CHRY_MX, K1E CHRY_MX, K1E2 CHRY_MX, K20 CHRY_MX, K21 CHRY_MX, K22 CHRY_MX, K23 CHRY_MX, K24 CHRY_MX, K25 CHRY_MX, K26 CHRY_MX, K27 CHRY_MX, K28 CHRY_MX, K29 CHRY_MX, K2A CHRY_MX, K2B CHRY_MX, K2C CHRY_MX, K30 CHRY_MX, K31 CHRY_MX, K32 CHRY_MX, K33 CHRY_MX, K34 CHRY_MX, K35 CHRY_MX, K36 CHRY_MX, K37 CHRY_MX, K38 CHRY_MX, K39 CHRY_MX, K3A CHRY_MX, K3B CHRY_MX, K3C CHRY_MX, K3E CHRY_MX, K3E2 CHRY_MX, K40 CHRY_MX, K402 CHRY_MX, K41 CHRY_MX, K42 CHRY_MX, K43 CHRY_MX, K44 CHRY_MX, K45 CHRY_MX, K46 CHRY_MX, K47 CHRY_MX, K48 CHRY_MX, K49 CHRY_MX, K4A CHRY_MX, K4B CHRY_MX, K4C CHRY_MX, K4D CHRY_MX, K4D2 CHRY_MX, K50 CHRY_MX, K51 CHRY_MX, K511 CHRY_MX, K52 CHRY_MX, K521 CHRY_MX, K53 CHRY_MX, K54 CHRY_MX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

Commit message: Release NKBM-ST110 r2.1 2018.05.08
Parts:
- removed the L07 at (220.8, 133.5)
- removed MODEL: NKBM-ST110_r2.0_18.02.11, null_keyboard:nkbm-st110_18.02
- added G***: LOGO, null_keyboard:nkbm-st110_18.05, F.Cu at (376.3, 125.0)
- added G***: LOGO, null_keyboard:nkbm-st110-silk_18.05, F.Cu at (376.2, 125.0)
- added K521: CHRY_MX, null_keyboard:CHERRY_PLATE_125H, F.Cu at (137.8, 167.3)
- added K521: CHRY_MX, null_keyboard:CHERRY_PLATE_125H, F.Cu at (159.2, 167.3)
- added K553: CHRY_MX, null_keyboard:CHERRY_PLATE_125H, F.Cu at (190.1, 167.3)
- added K572: CHRY_MX, null_keyboard:CHERRY_PLATE_125H, F.Cu at (211.7, 167.3)
- added K58: CHRY_MX, null_keyboard:CHERRY_PLATE_100H, F.Cu at (242.6, 167.3)
- added L07: LED, null_keyboard:LED_3MM, F.Cu at (263.8, 172.2)
- added L07: LED, null_keyboard:LED_3MM, F.Cu at (259.1, 172.2)
- added USB: Molex USB_Mini-B, Desktop:USB_Mini-B_Lumberg_2486_01_Horizontal, F.Cu at (414.5, 49.1)
- added USB DATA: BREAKOUT, null_keyboard:TEENSY2.0++, F.Cu at (424.9, 57.4)
- added USB POWER: BREAKOUT, null_keyboard:TEENSY2.0++, F.Cu at (404.6, 57.4)
- MCU1: value Teesny2.0++ -> Teesny++ 2.0
- moved R00 59.0 mm to (423.4, 75.2)
- moved R01 59.0 mm to (423.4, 78.7)
- moved R02 59.0 mm to (423.4, 81.9)
- moved L00 56.9 mm to (440.1, 74.7), turned to 0 degrees
- moved D06 56.6 mm to (180.8, 61.8)
- moved EXPANSION 56.6 mm to (449.9, 75.3)
- moved D07 56.5 mm to (199.8, 61.8)
- moved D66 56.5 mm to (356.9, 101.8)
- moved D60 56.4 mm to (355.2, 73.7)
- moved K6A 56.3 mm to (357.1, 167.3)
- moved D1E 56.3 mm to (333.0, 82.6)
- moved D5D 56.3 mm to (309.2, 156.7)
- moved D72 56.3 mm to (427.9, 111.4)
- moved D74 56.3 mm to (457.4, 100.7)
- moved K2C 56.3 mm to (304.5, 110.1)
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- renumbered RESET to RST
Routing:
- net /GND: track 831.9 -> 951.6 mm
- net /COL_07: track 658.9 -> 701.5 mm, vias 4 -> 3
- net (no net): track 0.00 -> 41.3 mm
- net Net-(D5E1-Pad1): track 6.08 -> 32.8 mm
- net /COL_09: track 429.9 -> 456.1 mm
- net /COL_14: track 621.7 -> 595.5 mm
- net /ROW_06: track 493.9 -> 471.5 mm, vias 4 -> 3
- net /COL_08: track 534.7 -> 557.1 mm
- net /COL_10: track 437.1 -> 417.8 mm, vias 2 -> 1
- net /COL_02: track 581.2 -> 599.9 mm
- net Net-(D091-Pad1): track 24.7 -> 6.83 mm
- net /LED_09: track 179.8 -> 166.7 mm
- net /LED_08: track 175.6 -> 162.5 mm
- net /COL_04: track 607.6 -> 619.6 mm, vias 4 -> 3
- net /RST: track 146.7 -> 158.6 mm
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Other:
- board size 426.8 x 121.9 mm -> 428.4 x 124.9 mm
- net class /GND: trace_width 1 -> 0.5; via_dia 0.5 -> 0.75
- net class Default: trace_width 1 -> 0.75; via_dia 0.5 -> 0.75
- net class Vbus added: clearance 0.3, trace_width 0.5, via_dia 0.75, via_drill 0.35
